Commit message: Updated sauce

File: src/x500_py/models/drone.urdf (robot description, URDF)
Before this commit: robot drone, 3 links, 2 joints
Links:
- link base_link: geometry visual mesh filename=file:///home/ros_workspace/src/x500_py/models/X500_drone.stl scale=1 1 1

Commit message: good sauce

File: src/x500_py/models/drone.urdf (robot description, URDF)
Before this commit: robot drone, 3 links, 2 joints
Links:
- link base_link: geometry visual mesh filename=file:///home/ros_workspace/src/x500_py/models/X500_drone_mo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 scale=1 1 1
